File: design_files/curl_tracker.kicad_pcb (KiCad board)
At the start: 2 copper layers, 50 x 60 mm, 55 parts, among them J1 JST-PH, J3 SSD1306 OLED, J4 JST-PH, J5 USB_C_Receptacle_USB2.0_16P, Q1 DMP2035, Q2 AO3400A, SW1 SW_Push, SW2 SW_Push, SW3 SW_Push, U1 TPS63001, U2 ESP32-C3-MINI-1, U3 MCP73831-2-OT, U4 BMI270, U5 USBLC6-2SC6

Commit message: finished pcb
Parts:
- moved C14 11.7 mm to (144.8, 90.0)
- moved C15 11.7 mm to (143.8, 90.0)
- moved U4 11.7 mm to (147.6, 90.0)
- moved R15 3.92 mm to (136.2, 102.0)
- moved Q2 3.77 mm to (133.4, 102.0)
- moved R16 3.76 mm to (133.4, 104.5)
- moved R17 3.01 mm to (160.7, 117.4), turned to 0 degrees
- moved SW3 2.03 mm to (157.6, 121.0)
- moved SW2 1.92 mm to (147.6, 121.0)
- moved SW1 1.91 mm to (137.6, 121.0), turned to 180 degrees
- moved C6 1.21 mm to (144.0, 80.0)
- moved J5 1.16 mm to (168.9, 86.6)
- moved R5 1.13 mm to (144.0, 78.7)
- moved J1 0.96 mm to (165.8, 106.6)
- moved J4 0.84 mm to (129.4, 96.6)
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Connections:
- net /USB_N renamed /D-
- net /USB_P renamed /D+
Routing:
- net +3.3V: track 18.5 -> 148.3 mm, vias 0 -> 12
- net Net-(U2-GPIO9): track 2.31 -> 67.0 mm, vias 0 -> 2
- net /IO5: track 0.00 -> 64.1 mm, vias 0 -> 4
- net Net-(U2-EN/CHIP_PU): track 4.49 -> 59.0 mm
- net VBATT: track 31.1 -> 74.7 mm
- net /IO3: track 0.00 -> 34.4 mm, vias 0 -> 4
- net /IO4: track 0.00 -> 32.4 mm, vias 0 -> 2
- net GND: track 58.4 -> 87.7 mm, vias 15 -> 46
- net /SDA: track 8.34 -> 33.6 mm
- net /SCL: track 8.07 -> 13.9 mm
- net Net-(U2-GPIO0/ADC1_CH0/XTAL_32K_P): track 0.00 -> 4.04 mm
- net /D+: track 14.7 -> 18.5 mm
- net /D-: track 16.7 -> 18.6 mm
- net Net-(J5-D--PadA7): track 5.97 -> 7.10 mm
- net Net-(J5-CC1): track 2.82 -> 3.84 mm
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- added copper zone on F.Cu, net GND
Other:
- board text added: "BATT"
- board text added: "BOOT"
- board text added: "DATA"
- board text added: "MOTOR"
- board text added: "RESET"
